File: MiniSTM32_ST7787_shield.sch (KiCad schematic (older format))
At the start: 6 parts, among them J1 CONN_02X16, J2 CONN_02X16, J3 CONN_02X12, U3 ET024002DMU

Commit message: WIP
work in progress
Parts:
- removed J1, J2: CONN_02X16, symbol CONN_02X16
- removed J3: CONN_02X12, symbol CONN_02X12
- added R0, R1: 0, Resistors_SMD:R_0805_HandSoldering, symbol R
- added U1: MiniSTM32F407, paccerlib:MiniSTM32F407_PinsRemoved, symbol MiniSTM32F407
- U3: footprint knielsenlib:ET024002DMU_otherside -> paccerlib:ET024002DMUrev2
- renumbered R8 to R2
Connections:
- net PC15 is gone; now on net +3V3: U3.2 (RESET)
- net +3V3: now also R1.2, U1.30 (3V3), U1.61 (3V3), U1.84 (3V3); no longer RV1.2
- net GND: now also U1.1 (GND), U1.29 (GND), U1.31 (GND), U1.34 (GND), U1.36 (GND), U1.62 (GND), U1.86 (GND)
- net PA0: now also U1.58 (PA0)
- net PA1: now also U1.55 (PA1)
- net PA10: now also U1.5 (PA10)
- net PA11: now also U1.8 (PA11)
- net PA12: now also U1.7 (PA12)
- net PA13: now also U1.10 (PA13)
- net PA14: now also U1.9 (PA14)
- net PA15: now also U1.12 (PA15)
- net PA2: now also U1.56 (PA2)
- net PA3: now also U1.54 (PA3)
- net PA4: now also U1.51 (PA4)
- net PA5: now also U1.52 (PA5)
- net PA6: now also U1.49 (PA6)
- net PA7: now also U1.50 (PA7)
- net PA8: now also U1.3 (PA8)
- net PA9: now also U1.6 (PA9)
- net PB0: now also U1.45 (PB0)
- net PB1: now also U1.46 (PB1)
- net PB10: now also U1.88 (PB10)
- net PB11: now also U1.85 (PB11)
- net PB12: now also U1.83 (PB12)
- net PB13: now also U1.82 (PB13)
- net PB14: now also U1.81 (PB14)
- net PB15: now also U1.80 (PB15)
- net PB2: now also U1.38 (PB2)
- net PB3: now also U1.24 (PB3)
- net PB4: now also U1.23 (PB4)
- net PB5: now also U1.26 (PB5)
- net PB6: now also U1.25 (PB6)
- net PB7: now also U1.28 (PB7)
- net PB8: now also U1.43 (PB8)
- net PB9: now also U1.44 (PB9)
- net PC0: now also U1.59 (PC0)
- net PC1: now also U1.60 (PC1)
- net PC10: now also U1.11 (PC10)
- net PC11: now also U1.14 (PC11)
- net PC12: now also U1.13 (PC12)
- net PC13: now also U1.64 (PC13)
- net PC2: now also U1.57 (PC2)
- net PC3: now also U1.53 (PC3)
- net PC4: now also U1.47 (PC4)
- net PC5: now also U1.48 (PC5)
- net PC6: now also U1.71 (PC6)
- net PC7: now also U1.70 (PC7)
- net PC8: now also U1.69 (PC8)
- net PC9: now also U1.4 (PC9)
- net PD0: now also U1.16 (PD0)
- net PD1: now also U1.15 (PD1)
- net PD10: now also U1.77 (PD10)
- net PD11: now also U1.76 (PD11)
- net PD12: now also U1.75 (PD12)
- net PD13: now also U1.74 (PD13)
- net PD14: now also U1.73 (PD14)
- net PD15: now also U1.72 (PD15)
- net PD2: now also U1.18 (PD2)
- net PD3: now also U1.17 (PD3)
- net PD4: now also U1.20 (PD4)
- net PD5: now also U1.19 (PD5)
- net PD6: now also U1.22 (PD6)
- net PD7: now also U1.21 (PD7)
- net PD8: now also U1.79 (PD8)
- net PD9: now also U1.78 (PD9)
- net PE0: now also U1.27 (PE0)
- net PE1: now also U1.41 (PE1)
- net PE10: now also U1.37 (PE10)
- net PE11: now also U1.91 (PE11)
- net PE12: now also U1.92 (PE12)
- net PE13: now also U1.89 (PE13)
- net PE14: now also U1.90 (PE14)
- net PE15: now also U1.87 (PE15)
- net PE2: now also U1.67 (PE2)
- net PE3: now also U1.68 (PE3)
- net PE4: now also U1.65 (PE4)
- net PE5: now also U1.66 (PE5)
- net PE6: now also U1.63 (PE6)
- net PE7: now also U1.42 (PE7)
- net PE8: now also U1.39 (PE8)
- net PE9: now also U1.40 (PE9)
- net VCC: now also R0.2, U1.2 (VCC), U1.32 (VCC)
- new net: R0.1, R1.1, RV1.2
- new net BOOT0: U1.35 (BOOT0)
- new net BOOT1: U1.33 (BOOT1)
- no-connect marks 77 -> 78
Other:
- note added: "backlight power source select"
- note removed: "todo:\n\nhardwire reset + check at det virker"
- moved on the sheet: R2, RV1, U3
